Commit message: habis ambil data parameter Q,R tgl 23-06

File: urdf/ackermann_edit.urdf.xacro (robot description, xacro)
@@ -12,5 +12,5 @@
     For this model:
     wheel_separation_h = base_length - front_center_offset - rear_center_offset = 0.15 -> wheelbase (harus 0.142)
-    wheel_separation_w = base_width  + 2 * axle_offset = 0.16 -> wheeltrack (harus 0.144)
+    wheel_separation_w = base_width  + 2 * axle_offset = 0.144 -> wheeltrack (harus 0.144)
 -->
 <robot name="ackermann_bot" xmlns:xacro="http://wiki.ros.org/xacro">
@@ -32,18 +32,18 @@
   <xacro:property name="deg_to_rad" value="0.01745329251994329577"/>
   <!-- Robot base dimensions -->
-  <xacro:property name="base_length" value="0.23" />
-  <xacro:property name="base_width" value="0.11" />
-  <xacro:property name="base_height" value="0.01" />
-  <xacro:property name="base_mass" value="133.5" />
+  <xacro:property name="base_length" value="0.222" />
+  <xacro:property name="base_width" value="0.12" />
+  <xacro:property name="base_height" value="0.03" />
+  <xacro:property name="base_mass" value="3" />
   <!-- Wheel link dimensions -->
-  <xacro:property name="wheel_radius" value="0.0375" />
+  <xacro:property name="wheel_radius" value="0.034" />
   <xacro:property name="wheel_thickness" value="0.025" />
-  <xacro:property name="wheel_mass" value="20" />
+  <xacro:property name="wheel_mass" value="0.25" />
   <!-- Steering link dimensions -->
   <xacro:property name="steer_radius" value="0.005" />
   <xacro:property name="steer_thickness" value="0.002" />
-  <xacro:property name="steer_mass" value="1" />
+  <xacro:property name="steer_mass" value="0.01" />
   <!-- Axle positions -->
-  <xacro:property name="axle_offset" value="0.025" />
+  <xacro:property name="axle_offset" value="0.012" />
   <xacro:property name="steer_offset" value="0.02" />
   <xacro:property name="front_center_offset" value="0.055" />
@@ -135,5 +135,5 @@
     wheel_radius="${wheel_radius}"
     wheel_thickness="${wheel_thickness}"
-    wheel_mass="${wheel_mass/12}">
+    wheel_mass="${wheel_mass}">
     <origin xyz="${-base_length/2+rear_center_offset} ${-base_width/2-axle_offset} 0" rpy="${-90 * deg_to_rad} 0 0"/>
   </xacro:rear_wheel_lr>
@@ -143,5 +143,5 @@
     wheel_radius="${wheel_radius}"
     wheel_thickness="${wheel_thickness}"
-    wheel_mass="${wheel_mass/12}">
+    wheel_mass="${wheel_mass}">
     <origin xyz="${-base_length/2+rear_center_offset} ${+base_width/2+axle_offset} 0" rpy="${-90 * deg_to_rad} 0 0"/>
   </xacro:rear_wheel_lr>
@@ -204,5 +204,5 @@
     <parent link="base_link"/>
     <child link="imu_link"/>
-    <origin xyz="0.0 0 0.2" rpy="0 0 ${-M_PI*0.5}"/>
+    <origin xyz="0.0 0 0.015" rpy="0 0 ${-M_PI*0.5}"/>
   </joint>
   <link name="imu_link"/>
